Commit message: fix: Updated materials and links
Updated the robot to use OGRE materials that will show in Gazebo
Also separated the links to apply materials to all links

Resolves comments from project review

File: my_robot/urdf/my_robot.xacro (robot description, xacro)
@@ -20,4 +20,10 @@
     <axis xyz="0 1 0"/>
   </joint>
+  <joint name="cab_joint" type="fixed">
+    <origin xyz="0 0 0" rpy="0 0 0"/>
+    <parent link="chassis"/>
+    <child link="cab" />
+    <axis xyz="0 1 0"/>
+  </joint>
   <joint name="front_right_wheel_hinge" type="continuous">
     <origin xyz="0.15 -0.15 0" rpy="0 0 0"/>
@@ -57,11 +63,29 @@
     <child link="arm_support" />
   </joint>
-  <joint name="arm_hinge" type="revolute">
+  <joint name="left_arm_hinge" type="revolute">
     <origin xyz="0 0 0" rpy="0 0 0"/>
     <parent link="arm_support"/>
-    <child link="arm"/>
+    <child link="left_arm"/>
     <axis xyz="0 1 0" rpy="0 0 0"/>
     <limit upper="0.52" lower="0" effort="10000" velocity="1000"/>
     <dynamics damping="1.0" friction="1.0"/>
+  </joint>
+  <joint name="right_arm_hinge" type="revolute">
+    <origin xyz="0 0 0" rpy="0 0 0"/>
+    <parent link="arm_support"/>
+    <child link="right_arm"/>
+    <axis xyz="0 1 0" rpy="0 0 0"/>
+    <limit upper="0.52" lower="0" effort="10000" velocity="1000"/>
+    <dynamics damping="1.0" friction="1.0"/>
+  </joint>
+  <joint name="right_bucket_hinge" type="fixed">
+    <origin xyz="0 0 0" rpy="0 0 0" />
+    <parent link="right_arm"/>
+    <child link="bucket" />
+  </joint>
+  <joint name="left_bucket_hinge" type="fixed">
+    <origin xyz="0 0 0" rpy="0 0 0" />
+    <parent link="left_arm"/>
+    <child link="bucket" />
   </joint>
   <!-- Links-->
@@ -90,18 +114,6 @@
       </geometry>
     </visual>
-    <collision name='cab_collision'>
-      <origin xyz="0.08 0 0.15" rpy=" 0 0 0"/>
-      <geometry>
-        <box size="0.3 0.18 0.3"/>
-      </geometry>
-    </collision>
-    <visual name='cab_visual'>
-      <origin xyz="0.08 0 0.15" rpy=" 0 0 0"/>
-      <geometry>
-        <box size="0.3 0.18 0.3"/>
-      </geometry>
-    </visual>
-  </link>
-  <link name='arm_support'>
+  </link>
+  <link name='cab'>
     <pose>0 0 0.1 0 0 0</pose>
     <inertial>
@@ -114,4 +126,28 @@
       />
     </inertial>
+    <collision name='cab_collision'>
+      <origin xyz="0.08 0 0.15" rpy=" 0 0 0"/>
+      <geometry>
+        <box size="0.3 0.18 0.3"/>
+      </geometry>
+    </collision>
+    <visual name='cab_visual'>
+      <origin xyz="0.08 0 0.15" rpy=" 0 0 0"/>
+      <geometry>
+        <box size="0.3 0.18 0.3"/>
+      </geometry>
+    </visual>
+  </link>
+  <link name='arm_support'>
+    <pose>0 0 0.1 0 0 0</pose>
+    <inertial>
+      <mass value="15.0"/>
+      <origin xyz="0.0 0 0" rpy=" 0 0 0"/>
+      <inertia
+          ixx="0.1" ixy="0" ixz="0"
+          iyy="0.1" iyz="0"
+          izz="0.1"
+      />
+    </inertial>
     <collision name='arm_support_collision'>
       <origin xyz="-0.15 0 0.15" rpy=" 0 0 0"/>
@@ -210,5 +246,5 @@
     </visual>
   </link>
-  <link name='arm'>
+  <link name='left_arm'>
      <inertial>
           <origin xyz="0.0 0 0" rpy="0 0 0"/>
@@ -230,4 +266,13 @@
       </geometry>
     </visual>
+  </link>
+  <link name='right_arm'>
+     <inertial>
+          <origin xyz="0.0 0 0" rpy="0 0 0"/>
+          <mass value="5.0"/>
+          <inertia ixx="0.1" ixy="0" ixz="0"
+                   iyy="0.1" iyz="0"
+                   izz="0.1"/>
+     </inertial>
     <collision name='right_arm_collision'>
       <origin xyz="0.08 -0.11 0.08" rpy="0 0.48 0"/>
@@ -242,4 +287,13 @@
       </geometry>
     </visual>
+  </link>
+  <link name='bucket'>
+     <inertial>
+          <origin xyz="0.0 0 0" rpy="0 0 0"/>
+          <mass value="5.0"/>
+          <inertia ixx="0.1" ixy="0" ixz="0"
+                   iyy="0.1" iyz="0"
+                   izz="0.1"/>
+     </inertial>
     <collision name='bucket_collision'>
       <origin xyz="0.36 0.1 0" rpy="0 0 0"/>
